File: pcb/Trabajo_Practico.sch (KiCad schematic (older format))
At the start: 42 parts, among them J1 USB_B_Micro, Q1 UMH3N, SW1 SW_MEC_5G, SW2 SW_SPDT, SW3 UP, SW4 DOWN, SW5 LEFT, SW6 RIGHT, SW7 A, SW8 B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

Commit message: Actualizacion de documentos y esquematico
Parts:
- added FID1, FID2, FID3: Fiducial, Fiducial:Fiducial_1.5mm_Mask3mm, symbol Mechanical:Fiducial
- added H1, H2, H3, H4: MountingHole, MountingHole:MountingHole_2.2mm_M2_Pad_Via, symbol Mechanical:MountingHole
- BT1: footprint (none) -> Battery:BatteryHolder_Keystone_2479_3xAAA; symbol Power_TP:Battery -> Components_TP:Battery
- BZ1: value Buzzer -> CMT-8503-85B-SMT-TR; footprint (none) -> TP_Footprints:MagneticBuzzer_CUI_CMT-8504-100-SMT; Mouser (none) -> https://ar.mouser.com/ProductDetail/CUI-Devices/CMT-8503-85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
- C1, C2, C3, C4, C5, C6: footprint (none) -> Capacitor_SMD:C_0805_2012Metric
- DS1: footprint (none) -> TP_Footprints:TFT_1.44I_SPI; symbol Display:ST7735_1.44_128x128_SPI -> Components_TP:ST7735_1.44_128x128_SPI
- F1: value Fuse_Small -> Fuse_Holder_Small; footprint (none) -> TP_Footprints:Fuse_Holder_Littefuse_Nano
- J1: footprint (none) -> Connector_USB:USB_Micro-B_Molex_47346-0001; Mouser (none) -> https://ar.mouser.com/ProductDetail/Amphenol-FCI/10104110-0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
- R1, R10, R11, R12, R13, R14, R15, R16, R17, R2, R3, R4, R5, R6, R7, R8, R9: footprint (none) -> Resistor_SMD:R_0805_2012Metric
- SW1: footprint (none) -> TP_Footprints:SW_Tactile_SPST_Angled_PTS645Vx31-2LFS
- SW2: footprint (none) -> Button_Switch_THT:SW_E-Switch_EG1224_SPDT_Angled
- SW3, SW4, SW5, SW6, SW7, SW8, SW9: footprint (none) -> TP_Footprints:SW_PUSH_6mm_H4.3mm
- U1: symbol Interface_USB_TP:CP2104 -> Components_TP:CP2104; Mouser (none) -> https://ar.mouser.com/ProductDetail/Silicon-Labs/CP2104-F03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
- U2: footprint (none) -> TP_Footprints:ESP-12E; symbol RF_Module_TP:ESP-12 -> Components_TP:ESP-12
- U3: footprint (none) -> Package_SO:TSSOP-24_4.4x7.8mm_P0.65mm; symbol Interface_Expansion_TP:PCA9539APW -> Components_TP:PCA9539APW; Mouser (none) -> https://ar.mouser.com/ProductDetail/NXP-Semiconductors/PCA9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
- U4: footprint (none) -> Package_TO_SOT_SMD:SOT-89-3_Handsoldering; symbol Regulator_Linear_TP:H7650-33PR -> Components_TP:H7650-33PR; Mouser (none) -> -
Connections:
- wire segments 196 -> 200
Other:
- note added: "Entradas Salidas"
- note added: "IC ST7735. La placa no cuenta con datasheet.\nSe coloca imagen de referencia."
- note added: "Se puede utilizar ESP12 / 12F / 12E /12S\nla diferencia radica en que cuenta con más pines de E/S, \npero no se utilizan en este circuito"
- note removed: "Expansion IO"
- note removed: "Ya que solo se cuenta con el integrado, \nse coloca imagen de referencia."
- moved on the sheet: BT1, BZ1, C1, C2, C5, C6, DS1, F1, J1, Q1A, Q1B, R8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

Commit message: Updated PCB component place and board edge
Parts:
- SW2: footprint Button_Switch_THT:SW_E-Switch_EG1224_SPDT_Angled -> Button_Switch_THT:SW_CuK_JS202011AQN_DPDT_Angled
Connections:
- net labels added: D+, D-
Changed lines of the file:
@@
 F 0 "SW2" H 8600 5135 50  0000 C CNN
 F 1 "SW_SPDT" H 8600 5044 50  0000 C CNN
-F 2 "Button_Switch_THT:SW_E-Switch_EG1224_SPDT_Angled" H 8600 4850 50  0001 C CNN
+F 2 "Button_Switch_THT:SW_CuK_JS202011AQN_DPDT_Angled" H 8600 4850 50  0001 C CNN
 F 3 "~" H 8600 4850 50  0001 C CNN
 	1    8600 4850
@@
 	1    0    0    -1
 $EndComp
+Text Label 1400 5800 0    50   ~ 0
+D+
+Text Label 1400 5900 0    50   ~ 0
+D-
 $EndSCHEMATC

Commit message: modified switch to SMD
Parts:
- SW3, SW4, SW5, SW6, SW7, SW8, SW9: footprint TP_Footprints:SW_PUSH_6mm_H4.3mm -> Button_Switch_SMD:SW_SPST_PTS645; symbol Switch:SW_MEC_5G -> Switch:SW_Push
Other:
- note added: "Impedancia controlada \n90 ohm diferencial"
Changed lines of the file:
@@
 	4000 2400 4000 2450
 $Comp
-L Switch:SW_MEC_5G SW3
+L Switch:SW_Push SW3
 U 1 1 61087190
 P 10350 1400
 F 0 "SW3" H 10200 1600 50  0000 C CNN
 F 1 "UP" H 10550 1600 50  0000 C CNN
-F 2 "TP_Footprints:SW_PUSH_6mm_H4.3mm" H 10350 1600 50  0001 C CNN
+F 2 "Button_Switch_SMD:SW_SPST_PTS645" H 10350 1600 50  0001 C CNN
 F 3 "http://www.apem.com/int/index.php?controller=attachment&id_attachment=488" H 10350 1600 50  0001 C CNN
 	1    10350 1400
@@
 $EndComp
 $Comp
-L Switch:SW_MEC_5G SW5
+L Switch:SW_Push SW5
 U 1 1 6108F321
 P 10350 2100
 F 0 "SW5" H 10200 2300 50  0000 C CNN
 F 1 "LEFT" H 10500 2300 50  0000 L CNN
-F 2 "TP_Footprints:SW_PUSH_6mm_H4.3mm" H 10350 2300 50  0001 C CNN
+F 2 "Button_Switch_SMD:SW_SPST_PTS645" H 10350 2300 50  0001 C CNN
 F 3 "http://www.apem.com/int/index.php?controller=attachment&id_attachment=488" H 10350 2300 50  0001 C CNN
 	1    10350 2100
@@
 $EndComp
 $Comp
-L Switch:SW_MEC_5G SW6
+L Switch:SW_Push SW6
 U 1 1 61097E28
 P 10350 2450
 F 0 "SW6" H 10200 2650 50  0000 C CNN
 F 1 "RIGHT" H 10600 2650 50  0000 C CNN
-F 2 "TP_Footprints:SW_PUSH_6mm_H4.3mm" H 10350 2650 50  0001 C CNN
+F 2 "Button_Switch_SMD:SW_SPST_PTS645" H 10350 2650 50  0001 C CNN
 F 3 "http://www.apem.com/int/index.php?controller=attachment&id_attachment=488" H 10350 2650 50  0001 C CNN
 	1    10350 2450
@@
 $EndComp
 $Comp
-L Switch:SW_MEC_5G SW7
+L Switch:SW_Push SW7
 U 1 1 6109AB65
 P 10350 2800
 F 0 "SW7" H 10200 3000 50  0000 C CNN
 F 1 "A" H 10550 3000 50  0000 C CNN
-F 2 "TP_Footprints:SW_PUSH_6mm_H4.3mm" H 10350 3000 50  0001 C CNN
+F 2 "Button_Switch_SMD:SW_SPST_PTS645" H 10350 3000 50  0001 C CNN
 F 3 "http://www.apem.com/int/index.php?controller=attachment&id_attachment=488" H 10350 3000 50  0001 C CNN
 	1    10350 2800
@@
 $EndComp
 $Comp
-L Switch:SW_MEC_5G SW9
+L Switch:SW_Push SW9
 U 1 1 610A0B8E
 P 10350 3500
 F 0 "SW9" H 10200 3700 50  0000 C CNN
 F 1 "C" H 10550 3700 50  0000 C CNN
-F 2 "TP_Footprints:SW_PUSH_6mm_H4.3mm" H 10350 3700 50  0001 C CNN
+F 2 "Button_Switch_SMD:SW_SPST_PTS645" H 10350 3700 50  0001 C CNN
 F 3 "http://www.apem.com/int/index.php?controller=attachment&id_attachment=488" H 10350 3700 50  0001 C CNN
 	1    10350 3500
@@
 	1300 5800 1700 5800
 $Comp
-L Connector:USB_B_Micro J1
-U 1 1 60E1A771
-P 1000 5800
-F 0 "J1" H 1057 6267 50  0000 C CNN
-F 1 "USB_B_Micro" H 1057 6176 50  0000 C CNN
-F 2 "Connector_USB:USB_Micro-B_Molex_47346-0001" H 1150 5750 50  0001 C CNN
-F 3 "~" H 1150 5750 50  0001 C CNN
-F 4 "https://ar.mouser.com/ProductDetail/Amphenol-FCI/10104110-0001LF?qs=%2Fha2pyFaduhgqo4mn6c%2FF%2F%2FdJtEtsNLYAPU1cSaXVJFvBbc5r%252BFA%252B%2FK9ZINccakG" H 1000 5800 50  0001 C CNN "Mouser"
-	1    1000 5800
-	1    0    0    -1
-$EndComp
-$Comp
 L Transistor_BJT:UMH3N Q1
 U 2 1 60E18F21
@@
 	10550 3500 10800 3500
 $Comp
-L Switch:SW_MEC_5G SW8
+L Switch:SW_Push SW8
 U 1 1 6109DAEE
 P 10350 3150
 F 0 "SW8" H 10200 3350 50  0000 C CNN
 F 1 "B" H 10550 3350 50  0000 C CNN
-F 2 "TP_Footprints:SW_PUSH_6mm_H4.3mm" H 10350 3350 50  0001 C CNN
+F 2 "Button_Switch_SMD:SW_SPST_PTS645" H 10350 3350 50  0001 C CNN
 F 3 "http://www.apem.com/int/index.php?controller=attachment&id_attachment=488" H 10350 3350 50  0001 C CNN
 	1    10350 3150
@@
 	9550 2450 10150 2450
 $Comp
-L Switch:SW_MEC_5G SW4
+L Switch:SW_Push SW4
 U 1 1 6108A64D
 P 10350 1750
 F 0 "SW4" H 10200 1950 50  0000 C CNN
 F 1 "DOWN" H 10600 1950 50  0000 C CNN
-F 2 "TP_Footprints:SW_PUSH_6mm_H4.3mm" H 10350 1950 50  0001 C CNN
+F 2 "Button_Switch_SMD:SW_SPST_PTS645" H 10350 1950 50  0001 C CNN
 F 3 "http://www.apem.com/int/index.php?controller=attachment&id_attachment=488" H 10350 1950 50  0001 C CNN
 	1    10350 1750
@@
 Text Label 1400 5900 0    50   ~ 0
 D-
+Text Notes 550  6750 0    50   ~ 0
+Impedancia controlada \n90 ohm diferencial
+$Comp
+L Connector:USB_B_Micro J1
+U 1 1 60E1A771
+P 1000 5800
+F 0 "J1" H 1057 6267 50  0000 C CNN
+F 1 "USB_B_Micro" H 1057 6176 50  0000 C CNN
+F 2 "Connector_USB:USB_Micro-B_Molex_47346-0001" H 1150 5750 50  0001 C CNN
+F 3 "~" H 1150 5750 50  0001 C CNN
+F 4 "https://ar.mouser.com/ProductDetail/Amphenol-FCI/10104110-0001LF?qs=%2Fha2pyFaduhgqo4mn6c%2FF%2F%2FdJtEtsNLYAPU1cSaXVJFvBbc5r%252BFA%252B%2FK9ZINccakG" H 1000 5800 50  0001 C CNN "Mouser"
+	1    1000 5800
+	1    0    0    -1
+$EndComp
+Wire Notes Line
+	1550 5750 1550 6550
+Wire Notes Line
+	1550 6550 1350 6750
+Wire Notes Line
+	550  6750 1350 6750
 $EndSCHEMATC

Commit message: Routed and checked
Parts:
- BZ1: Mouser https://ar.mouser.com/ProductDetail/CUI-Devices/CMT-8503-85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 -> 490-CMT-850385BSMTTR; Mouser Link (none) -> https://ar.mouser.com/ProductDetail/CUI-Devices/CMT-8503-85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
- J1: Mouser https://ar.mouser.com/ProductDetail/Amphenol-FCI/10104110-0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 -> 649-10104110-0001LF; Mouser Link (none) -> https://ar.mouser.com/ProductDetail/Amphenol-FCI/10104110-0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
- Q1: Mouser (none) -> 755-UMH3NFHATN; Mouser Link (none) -> https://ar.mouser.com/ProductDetail/ROHM-Semiconductor/UMH3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
- U1: Mouser https://ar.mouser.com/ProductDetail/Silicon-Labs/CP2104-F03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 -> 634-CP2104-F03-GM; Mouser Link (none) -> https://ar.mouser.com/ProductDetail/Silicon-Labs/CP2104-F03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
- U3: Mouser https://ar.mouser.com/ProductDetail/NXP-Semiconductors/PCA9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 -> 771-PCA9539APW,118; Mouser Link (none) -> https://ar.mouser.com/ProductDetail/NXP-Semiconductors/PCA9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
Other:
- moved on the sheet: SW4, SW5, SW6
Changed lines of the file:
@@
 F 2 "Package_SO:TSSOP-24_4.4x7.8mm_P0.65mm" H 6800 3600 50  0001 C CNN
 F 3 "https://www.nxp.com/docs/en/data-sheet/PCA9539A.pdf" H 6800 3600 50  0001 C CNN
-F 4 "https://ar.mouser.com/ProductDetail/NXP-Semiconductors/PCA9539APW118?qs=%2Fha2pyFaduh%2Fi8YhwVy9WcgkUZjuwavpcMUMzd3dW5Ablgd5XfULPA%3D%3D" H 7200 2550 50  0001 C CNN "Mouser"
+F 4 "https://ar.mouser.com/ProductDetail/NXP-Semiconductors/PCA9539APW118?qs=%2Fha2pyFaduh%2Fi8YhwVy9WcgkUZjuwavpcMUMzd3dW5Ablgd5XfULPA%3D%3D" H 7200 2550 50  0001 C CNN "Mouser Link"
+F 5 "771-PCA9539APW,118" H 7200 2550 50  0001 C CNN "Mouser"
 	1    7200 2550
 	1    0    0    -1
@@
 F 2 "TP_Footprints:ESP-12E" H 2600 2650 50  0001 C CNN
 F 3 "https://www.elecrow.com/download/ESP-12S_User_Manual.pdf" H 2600 2650 50  0001 C CNN
+F 4 "" H 3050 2050 50  0001 C CNN "Mouser Link"
+F 5 "" H 3050 2050 50  0001 C CNN "Mouser"
 	1    3050 2050
 	1    0    0    -1
 $EndComp
 $Comp
-L Components_TP:H7650-33PR U4
-U 1 1 60E16F0A
-P 10050 4850
-F 0 "U4" H 10050 5092 50  0000 C CNN
-F 1 "H7650-33PR" H 10050 5001 50  0000 C CNN
-F 2 "Package_TO_SOT_SMD:SOT-89-3_Handsoldering" H 9800 5000 50  0001 C CNN
-F 3 "https://xonstorage.blob.core.windows.net/pdf/siproin_h765033pr_Lcs01_link.pdf" H 9800 5000 50  0001 C CNN
-F 4 "-" H 10050 4850 50  0001 C CNN "Mouser"
-	1    10050 4850
-	1    0    0    -1
-$EndComp
-$Comp
 L Switch:SW_SPDT SW2
 U 1 1 60E242D5
@@
 L Switch:SW_Push SW5
 U 1 1 6108F321
-P 10350 2100
-F 0 "SW5" H 10200 2300 50  0000 C CNN
-F 1 "LEFT" H 10500 2300 50  0000 L CNN
-F 2 "Button_Switch_SMD:SW_SPST_PTS645" H 10350 2300 50  0001 C CNN
-F 3 "http://www.apem.com/int/index.php?controller=attachment&id_attachment=488" H 10350 2300 50  0001 C CNN
-	1    10350 2100
+P 10350 1750
+F 0 "SW5" H 10200 1950 50  0000 C CNN
+F 1 "LEFT" H 10500 1950 50  0000 L CNN
+F 2 "Button_Switch_SMD:SW_SPST_PTS645" H 10350 1950 50  0001 C CNN
+F 3 "http://www.apem.com/int/index.php?controller=attachment&id_attachment=488" H 10350 1950 50  0001 C CNN
+	1    10350 1750
 	1    0    0    -1
 $EndComp
@@
 L Switch:SW_Push SW6
 U 1 1 61097E28
-P 10350 2450
-F 0 "SW6" H 10200 2650 50  0000 C CNN
-F 1 "RIGHT" H 10600 2650 50  0000 C CNN
-F 2 "Button_Switch_SMD:SW_SPST_PTS645" H 10350 2650 50  0001 C CNN
-F 3 "http://www.apem.com/int/index.php?controller=attachment&id_attachment=488" H 10350 2650 50  0001 C CNN
-	1    10350 2450
+P 10350 2100
+F 0 "SW6" H 10200 2300 50  0000 C CNN
+F 1 "RIGHT" H 10600 2300 50  0000 C CNN
+F 2 "Button_Switch_SMD:SW_SPST_PTS645" H 10350 2300 50  0001 C CNN
+F 3 "http://www.apem.com/int/index.php?controller=attachment&id_attachment=488" H 10350 2300 50  0001 C CNN
+	1    10350 2100
 	1    0    0    -1
 $EndComp
@@
 F 2 "TP_Footprints:MagneticBuzzer_CUI_CMT-8504-100-SMT" V 5325 2300 50  0001 C CNN
 F 3 "https://ar.mouser.com/datasheet/2/670/cmt_8503_85b_smt_tr-1777166.pdf" V 5325 2300 50  0001 C CNN
-F 4 "https://ar.mouser.com/ProductDetail/CUI-Devices/CMT-8503-85B-SMT-TR?qs=P1JMDcb91o7ndeE%252B1xd5mQ%3D%3D" H 5350 2200 50  0001 C CNN "Mouser"
+F 4 "https://ar.mouser.com/ProductDetail/CUI-Devices/CMT-8503-85B-SMT-TR?qs=P1JMDcb91o7ndeE%252B1xd5mQ%3D%3D" H 5350 2200 50  0001 C CNN "Mouser Link"
+F 5 "490-CMT-850385BSMTTR" H 5350 2200 50  0001 C CNN "Mouser"
 	1    5350 2200
 	1    0    0    -1
@@
 F 2 "Package_TO_SOT_SMD:SOT-363_SC-70-6" H 4005 5860 50  0001 C CNN
 F 3 "http://rohmfs.rohm.com/en/products/databook/datasheet/discrete/transistor/digital/emh3t2r-e.pdf" H 4150 6300 50  0001 C CNN
+F 4 "755-UMH3NFHATN" V 4000 6300 50  0001 C CNN "Mouser"
+F 5 "https://ar.mouser.com/ProductDetail/ROHM-Semiconductor/UMH3NFHATN?qs=4v%252BiZTmLVHETwyIExWQvig%3D%3D" V 4000 6300 50  0001 C CNN "Mouser Link"
 	2    4000 6300
 	0    1    1    0
@@
 F 2 "Package_TO_SOT_SMD:SOT-363_SC-70-6" H 4005 5060 50  0001 C CNN
 F 3 "http://rohmfs.rohm.com/en/products/databook/datasheet/discrete/transistor/digital/emh3t2r-e.pdf" H 4150 5500 50  0001 C CNN
+F 4 "755-UMH3NFHATN" V 4000 5500 50  0001 C CNN "Mouser"
+F 5 "https://ar.mouser.com/ProductDetail/ROHM-Semiconductor/UMH3NFHATN?qs=4v%252BiZTmLVHETwyIExWQvig%3D%3D" V 4000 5500 50  0001 C CNN "Mouser Link"
 	1    4000 5500
 	0    1    1    0
@@
 F 2 "Package_DFN_QFN:QFN-24-1EP_4x4mm_P0.5mm_EP2.6x2.6mm" H 2550 5100 50  0001 L CNN
 F 3 "https://www.silabs.com/documents/public/data-sheets/cp2104.pdf" H 1850 7300 50  0001 C CNN
-F 4 "https://ar.mouser.com/ProductDetail/Silicon-Labs/CP2104-F03-GM?qs=j12q4iUN960zrcKDk%2FjKbw%3D%3D" H 2400 6050 50  0001 C CNN "Mouser"
+F 4 "https://ar.mouser.com/ProductDetail/Silicon-Labs/CP2104-F03-GM?qs=j12q4iUN960zrcKDk%2FjKbw%3D%3D" H 2400 6050 50  0001 C CNN "Mouser Link"
+F 5 "634-CP2104-F03-GM" H 2400 6050 50  0001 C CNN "Mouser"
 	1    2400 6050
 	1    0    0    -1
@@
 L Switch:SW_Push SW4
 U 1 1 6108A64D
-P 10350 1750
-F 0 "SW4" H 10200 1950 50  0000 C CNN
-F 1 "DOWN" H 10600 1950 50  0000 C CNN
-F 2 "Button_Switch_SMD:SW_SPST_PTS645" H 10350 1950 50  0001 C CNN
-F 3 "http://www.apem.com/int/index.php?controller=attachment&id_attachment=488" H 10350 1950 50  0001 C CNN
-	1    10350 1750
+P 10350 2450
+F 0 "SW4" H 10200 2650 50  0000 C CNN
+F 1 "DOWN" H 10600 2650 50  0000 C CNN
+F 2 "Button_Switch_SMD:SW_SPST_PTS645" H 10350 2650 50  0001 C CNN
+F 3 "http://www.apem.com/int/index.php?controller=attachment&id_attachment=488" H 10350 2650 50  0001 C CNN
+	1    10350 2450
 	1    0    0    -1
 $EndComp
@@
 Text Notes 550  6750 0    50   ~ 0
 Impedancia controlada \n90 ohm diferencial
+Wire Notes Line
+	1550 5750 1550 6550
+Wire Notes Line
+	1550 6550 1350 6750
+Wire Notes Line
+	550  6750 1350 6750
 $Comp
 L Connector:USB_B_Micro J1
@@
 F 1 "USB_B_Micro" H 1057 6176 50  0000 C CNN
 F 2 "Connector_USB:USB_Micro-B_Molex_47346-0001" H 1150 5750 50  0001 C CNN
-F 3 "~" H 1150 5750 50  0001 C CNN
-F 4 "https://ar.mouser.com/ProductDetail/Amphenol-FCI/10104110-0001LF?qs=%2Fha2pyFaduhgqo4mn6c%2FF%2F%2FdJtEtsNLYAPU1cSaXVJFvBbc5r%252BFA%252B%2FK9ZINccakG" H 1000 5800 50  0001 C CNN "Mouser"
+F 3 "https://www.amphenol-icc.com/media/wysiwyg/files/documentation/datasheet/inputoutput/io_usb_micro.pdf" H 1150 5750 50  0001 C CNN
+F 4 "https://ar.mouser.com/ProductDetail/Amphenol-FCI/10104110-0001LF?qs=%2Fha2pyFaduhgqo4mn6c%2FF%2F%2FdJtEtsNLYAPU1cSaXVJFvBbc5r%252BFA%252B%2FK9ZINccakG" H 1000 5800 50  0001 C CNN "Mouser Link"
+F 5 "649-10104110-0001LF" H 1000 5800 50  0001 C CNN "Mouser"
 	1    1000 5800
 	1    0    0    -1
 $EndComp
-Wire Notes Line
-	1550 5750 1550 6550
-Wire Notes Line
-	1550 6550 1350 6750
-Wire Notes Line
-	550  6750 1350 6750
+$Comp
+L Components_TP:H7650-33PR U4
+U 1 1 60E16F0A
+P 10050 4850
+F 0 "U4" H 10050 5092 50  0000 C CNN
+F 1 "H7650-33PR" H 10050 5001 50  0000 C CNN
+F 2 "Package_TO_SOT_SMD:SOT-89-3_Handsoldering" H 9800 5000 50  0001 C CNN
+F 3 "https://xonstorage.blob.core.windows.net/pdf/siproin_h765033pr_Lcs01_link.pdf" H 9800 5000 50  0001 C CNN
+F 4 "-" H 10050 4850 50  0001 C CNN "Mouser"
+	1    10050 4850
+	1    0    0    -1
+$EndComp
 $EndSCHEMATC
